Commit message: fixed issues for SLAM obstacle spawning

File: description/urdf/sensors.xacro (robot description, xacro)
@@ -2,4 +2,107 @@
 <!-- Sherpa Sensors-->
 <robot name ="sherpa_sensors" xmlns:xacro="http://www.ros.org/wiki/xacro">
+	<!-- Rear left sick sensor -->
+  	<link name="rear_sick">
+        <visual>
+            <geometry>
+                <cylinder radius="0.05" length="0.12"/>
+            </geometry>
+            <origin xyz="0 0 0" rpy="0 0 0"/>
+        </visual>
+        <inertial>
+            <origin xyz="0 0 0" rpy="0 0 0"/>
+	        <mass value="1.0" />
+	        <inertia  ixx="1.0" ixy="0.0" ixz="0.0" iyy="1.0" iyz="0.0" izz="1.0"/>
+	     </inertial>
+  	</link>
+    <gazebo reference="rear_sick"><material>Gazebo/Yellow</material></gazebo>
+    <joint name="rear_sick_to_chassis" type="fixed">
+        <parent link="chassis"/>
+        <child link="rear_sick"/>
+        <origin xyz="-0.8775 0.5225 0.35" rpy="3.1415 0 2.35619"/>
+    </joint>
+	<gazebo reference="rear_sick">
+		<sensor type="ray" name="rear_sick_sensor">
+			<pose>0 0 0 0 0 0</pose>
+			<visualize>true</visualize>
+			<update_rate>12</update_rate>
+			<ray>
+				<scan>
+					<horizontal>
+						<samples>761</samples>
+						<resolution>1</resolution>
+						<min_angle>-2.356195</min_angle>
+						<max_angle>2.356195</max_angle>
+					</horizontal>
+				</scan>
+				<range>
+					<min>0.10</min>
+					<max>8.0</max>
+					<resolution>0.01</resolution>
+				</range>
+				<noise>
+					<type>gaussian</type>
+					<mean>0.0</mean>
+					<stddev>0.01</stddev>
+				</noise>
+			</ray>
+			<plugin name="sick_controller" filename="libgazebo_ros_laser.so">
+				<topicName>/rear_sick/scan</topicName>
+				<frameName>rear_sick</frameName>
+			</plugin>
+		</sensor>
+	</gazebo>
+	<!-- Front right sick sensor -->
+  	<link name="front_sick">
+        <visual>
+            <geometry>
+                <cylinder radius="0.05" length="0.12"/>
+            </geometry>
+            <origin xyz="0 0 0" rpy="0 0 0"/>
+        </visual>
+        <inertial>
+            <origin xyz="0 0 0" rpy="0 0 0"/>
+	        <mass value="1.0" />
+	        <inertia  ixx="1.0" ixy="0.0" ixz="0.0" iyy="1.0" iyz="0.0" izz="1.0"/>
+	     </inertial>
+  </link>
+    <gazebo reference="front_sick"><material>Gazebo/Yellow</material></gazebo>
+    <joint name="front_sick_to_chassis" type="fixed">
+        <parent link="chassis"/>
+        <child link="front_sick"/>
+        <origin xyz="0.8775 -0.5225 0.35" rpy="3.1415 0 -0.785398"/>
+    </joint>
+    <gazebo reference="front_sick">
+			<sensor type="ray" name="front_sick_sensor">
+				<pose>0 0 0 0 0 0</pose>
+				<visualize>true</visualize>
+				<update_rate>12</update_rate>
+				<ray>
+					<scan>
+						<horizontal>
+							<samples>761</samples>
+							<resolution>1</resolution>
+							<min_angle>-2.356195</min_angle>
+							<max_angle>2.356195</max_angle>
+						</horizontal>
+					</scan>
+					<range>
+						<min>0.10</min>
+						<max>8.0</max>
+						<resolution>0.01</resolution>
+					</range>
+					<noise>
+						<type>gaussian</type>
+						<mean>0.0</mean>
+						<stddev>0.01</stddev>
+					</noise>
+				</ray>
+				<plugin name="sick_controller" filename="libgazebo_ros_laser.so">
+					<topicName>/front_sick/scan</topicName>
+					<frameName>front_sick</frameName>
+				</plugin>
+			</sensor>
+		</gazebo>
+</robot>
 <!--link name="imu_link">
         <visual>
@@ -40,106 +143,4 @@
     	</sensor>
   	</gazebo-->
-  <!-- Front right sick sensor -->
-  <link name="front_sick">
-        <visual>
-            <geometry>
-                <cylinder radius="0.05" length="0.12"/>
-            </geometry>
-            <origin xyz="0 0 0" rpy="0 0 0"/>
-        </visual>
-        <inertial>
-            <origin xyz="0 0 0" rpy="0 0 0"/>
-	        <mass value="1.0" />
-	        <inertia  ixx="1.0" ixy="0.0" ixz="0.0" iyy="1.0" iyz="0.0" izz="1.0"/>
-	     </inertial>
-  </link>
-      <gazebo reference="front_sick"><material>Gazebo/Yellow</material></gazebo>
-    <joint name="front_sick_to_chassis" type="fixed">
-        <parent link="chassis"/>
-        <child link="front_sick"/>
-        <origin xyz="0.8775 -0.5225 0.35" rpy="3.1415 0 -0.785398"/>
-    </joint>
-    <gazebo reference="front_sick">
-			<sensor type="ray" name="front_sick_sensor">
-				<pose>0 0 0 0 0 0</pose>
-				<visualize>false</visualize>
-				<update_rate>16.6</update_rate>
-				<ray>
-					<scan>
-						<horizontal>
-							<samples>761</samples>
-							<resolution>1</resolution>
-							<min_angle>-2.356195</min_angle>
-							<max_angle>2.356195</max_angle>
-						</horizontal>
-					</scan>
-					<range>
-						<min>0.10</min>
-						<max>9.0</max>
-						<resolution>0.01</resolution>
-					</range>
-					<noise>
-						<type>gaussian</type>
-						<mean>0.0</mean>
-						<stddev>0.01</stddev>
-					</noise>
-				</ray>
-				<plugin name="sick_controller" filename="libgazebo_ros_laser.so">
-					<topicName>/scan</topicName>
-					<frameName>front_sick</frameName>
-				</plugin>
-			</sensor>
-		</gazebo>
-		<!-- Rear left sick sensor -->
-  <link name="rear_sick">
-        <visual>
-            <geometry>
-                <cylinder radius="0.05" length="0.12"/>
-            </geometry>
-            <origin xyz="0 0 0" rpy="0 0 0"/>
-        </visual>
-        <inertial>
-            <origin xyz="0 0 0" rpy="0 0 0"/>
-	        <mass value="1.0" />
-	        <inertia  ixx="1.0" ixy="0.0" ixz="0.0" iyy="1.0" iyz="0.0" izz="1.0"/>
-	     </inertial>
-  </link>
-      <gazebo reference="rear_sick"><material>Gazebo/Yellow</material></gazebo>
-    <joint name="rear_sick_to_chassis" type="fixed">
-        <parent link="chassis"/>
-        <child link="rear_sick"/>
-        <origin xyz="-0.8775 0.5225 0.35" rpy="3.1415 0 2.35619"/>
-    </joint>
-       <gazebo reference="rear_sick">
-			<sensor type="ray" name="rear_sick_sensor">
-				<pose>0 0 0 0 0 0</pose>
-				<visualize>false</visualize>
-				<update_rate>16.6</update_rate>
-				<ray>
-					<scan>
-						<horizontal>
-							<samples>761</samples>
-							<resolution>1</resolution>
-							<min_angle>-2.356195</min_angle>
-							<max_angle>2.356195</max_angle>
-						</horizontal>
-					</scan>
-					<range>
-						<min>0.10</min>
-						<max>9.0</max>
-						<resolution>0.01</resolution>
-					</range>
-					<noise>
-						<type>gaussian</type>
-						<mean>0.0</mean>
-						<stddev>0.01</stddev>
-					</noise>
-				</ray>
-				<plugin name="sick_controller" filename="libgazebo_ros_laser.so">
-					<topicName>/scan</topicName>
-					<frameName>rear_sick</frameName>
-				</plugin>
-			</sensor>
-		</gazebo>
 		<!-- Velodyne sensor -->
 <!--		<link name="velodyne_base">-->
@@ -226,3 +227,2 @@
 <!--			</sensor>-->
 <!--		</gazebo>-->
-</robot>

File: description/urdf/sherpa_ros_ackermann.xacro (robot description, xacro)
@@ -169,6 +169,4 @@
         <fake_inertial/>
     </link>
-<!-->xacro:include filename="sprayer.xacro"/-->
-<xacro:include filename="sensors.xacro"/>
   <gazebo>
     <plugin name="ground_truth" filename="libgazebo_ros_p3d.so">
@@ -182,8 +180,9 @@
       <rpyOffsets>0 0 0</rpyOffsets>
     </plugin>
-<!-- ros_control plugin -->
+    <!-- ros_control plugin -->
     <plugin name="gazebo_ros_control" filename="libgazebo_ros_control.so">
           <legacyModeNS>true</legacyModeNS>
           </plugin>
   </gazebo>
+  <xacro:include filename="sensors.xacro"/>
 </robot>

File: description/urdf/sherpa_ros_omni.xacro (robot description, xacro)
@@ -119,5 +119,4 @@
 <!-- Include sherpa_wheel.xacro file -->
 <xacro:include filename="sherpa_wheel_omni.xacro"/>
-<xacro:include filename="sensors.xacro"/>
 <xacro:include filename="torso.xacro"/>
 <xacro:include filename="gun.xacro"/>

Commit message: omni model fix and multi global planner

File: description/urdf/sensors.xacro (robot description, xacro)
@@ -2,4 +2,5 @@
 <!-- Sherpa Sensors-->
 <robot name ="sherpa_sensors" xmlns:xacro="http://www.ros.org/wiki/xacro">
+	<xacro:arg name="velodyne_enabled" default="false"/>
 	<!-- Rear left sick sensor -->
   	<link name="rear_sick">
@@ -25,5 +26,5 @@
 		<sensor type="ray" name="rear_sick_sensor">
 			<pose>0 0 0 0 0 0</pose>
-			<visualize>true</visualize>
+			<visualize>false</visualize>
 			<update_rate>12</update_rate>
 			<ray>
@@ -76,5 +77,5 @@
 			<sensor type="ray" name="front_sick_sensor">
 				<pose>0 0 0 0 0 0</pose>
-				<visualize>true</visualize>
+				<visualize>false</visualize>
 				<update_rate>12</update_rate>
 				<ray>
@@ -104,4 +105,95 @@
 			</sensor>
 		</gazebo>
+    <!-- Velodye -->
+	<joint name="velodyne_joint" type="fixed">
+		<parent link="chassis"/>
+		<child link="velodyne_base_link"/>
+		<origin xyz="0.8815 0.0 0.3334" rpy="0 0 0"/> <!-- Inserire inclinazione del velodyne -->
+	</joint>
+	<link name="velodyne_base_link">
+      <inertial>
+        <mass value="0.83"/>
+        <origin xyz="0 0 0.03585"/>
+        <inertia ixx="${(0.83 * (3.0*0.0516*0.0516 + 0.0717*0.0717)) / 12.0}" ixy="0" ixz="0"
+          iyy="${(0.83 * (3.0*0.0516*0.0516 + 0.0717*0.0717)) / 12.0}" iyz="0"
+          izz="${0.5 * 0.83 * (0.0516*0.0516)}"/>
+      </inertial>
+      <visual>
+        <geometry>
+          <mesh filename="package://velodyne_description/meshes/VLP16_base_1.dae" />
+        </geometry>
+      </visual>
+      <visual>
+        <geometry>
+          <mesh filename="package://velodyne_description/meshes/VLP16_base_2.dae" />
+        </geometry>
+      </visual>
+      <collision>
+        <origin rpy="0 0 0" xyz="0 0 0.03585"/>
+        <geometry>
+          <cylinder radius="0.0516" length="0.0717"/>
+        </geometry>
+      </collision>
+    </link>
+    <joint name="velodyne_base_scan_joint" type="fixed" >
+      <origin xyz="0 0 0.0377" rpy="0 0 0" />
+      <parent link="velodyne_base_link" />
+      <child link="velodyne"/>
+    </joint>
+    <link name="velodyne">
+      <inertial>
+        <mass value="0.01"/>
+        <origin xyz="0 0 0"/>
+        <inertia ixx="1e-7" ixy="0" ixz="0" iyy="1e-7" iyz="0" izz="1e-7"/>
+      </inertial>
+      <visual>
+        <origin xyz="0 0 -0.0377" />
+        <geometry>
+          <mesh filename="package://velodyne_description/meshes/VLP16_scan.dae" />
+        </geometry>
+      </visual>
+    </link>
+	<xacro:if value="$(arg velodyne_enabled)">
+	<gazebo reference="velodyne">
+		<sensor type="ray" name="VLP16">
+			<pose>0 0 0 0 0 0</pose>
+			<visualize>true</visualize>
+			<update_rate>10</update_rate>
+			<ray>
+				<scan>
+						<horizontal>
+							<samples>360</samples>
+							<resolution>1</resolution>
+							<min_angle>-${PI}</min_angle>
+							<max_angle> ${PI}</max_angle>
+						</horizontal>
+					<vertical>
+						<samples>16</samples>
+						<resolution>1</resolution>
+						<min_angle>-${15.0*PI/180.0}</min_angle>
+						<max_angle> ${15.0*PI/180.0}</max_angle>
+					</vertical>
+				</scan>
+				<range>
+					<min>0.3</min>
+					<max>131.0</max>
+					<resolution>0.001</resolution>
+				</range>
+				<noise>
+					<type>gaussian</type>
+					<mean>0.0</mean>
+					<stddev>0.0</stddev>
+				</noise>
+			</ray>
+			<plugin name="gazebo_ros_laser_controller" filename="libgazebo_ros_velodyne_laser.so">
+				<topicName>velodyne_points</topicName>
+				<frameName>velodyne</frameName>
+				<min_range>1.0</min_range>
+				<max_range>140.0</max_range>
+				<gaussianNoise>0.008</gaussianNoise>
+			</plugin>
+		</sensor>
+	</gazebo>
+	</xacro:if>
 </robot>
 <!--link name="imu_link">

File: description/urdf/sherpa_ros_ackermann.xacro (robot description, xacro)
@@ -2,6 +2,6 @@
 <!-- Sherpa -->
 <robot name ="sherpa" xmlns:xacro="http://www.ros.org/wiki/xacro">
-<!-- Parameters -->
-<xacro:property name="PI" value="3.1415926535897931"/>
+  <!-- Parameters -->
+  <xacro:property name="PI" value="3.1415926535897931"/>
   <!-- Chassis Property -->
   <xacro:property name="chassis_x" value="0.8275"/>

File: description/urdf/sherpa_ros_omni-ackermann.xacro (robot description, xacro)
@@ -69,5 +69,5 @@
     <parent link="base_link"/>
     <child link="chassis"/>
-    <origin xyz="0 0 0"/>
+    <origin xyz="0.667 0 0"/>
   </joint>
   <!-- Chassis -->
@@ -119,15 +119,15 @@
   <gazebo reference="cable_box"><material>Gazebo/Red</material></gazebo>
 <!-- Include sherpa_wheel.xacro file -->
-<xacro:include filename="sherpa_wheel_omni.xacro"/>
-<xacro:include filename="torso.xacro"/>
-<xacro:include filename="gun.xacro"/>
+<xacro:include filename="sherpa_wheel_omni-ackermann.xacro"/>
+<xacro:include filename="torso_omni-ackermann.xacro"/>
+<xacro:include filename="gun_omni-ackermann.xacro"/>
   <gazebo>
     <plugin name="ground_truth" filename="libgazebo_ros_p3d.so">
       <alwaysOn>true</alwaysOn>
-      <updateRate>50.0</updateRate>
+      <updateRate>100.0</updateRate>
       <bodyName>base_link</bodyName>
-      <topicName>/odom_gps</topicName>
+      <topicName>odom_gps</topicName>
       <gaussianNoise>0.00</gaussianNoise>
-      <frameName>map</frameName>
+      <frameName>/map</frameName>
       <xyzOffsets>0 0 0</xyzOffsets>
       <rpyOffsets>0 0 0</rpyOffsets>
